Commit message: Add Fishbot navigation and simulation package with URDF and Gazebo configuration

File: chap_navigation/src/demo_description/urdf/fishbot/sensor/imu.urdf.xacro (robot description, xacro)
@@ -2,12 +2,16 @@
 <robot xmlns:xacro="http://ros.org/wiki/xacro" >
     <xacro:include filename="$(find demo_description)/urdf/fishbot/common_inertia.xacro"/>
-    <xacro:macro name="camera_link" params="xyz">
+    <xacro:macro name="imu_link" params="xyz">
             <!-- 机器人的IMU部件，惯性测量传感器 -->
-        <link name="camera_link">
+        <link name="imu_link">
             <visual>
+                <!-- 沿着自己几何中心的偏移和旋转量 -->
                 <origin xyz="0 0 0" rpy="0 0 0"/>
+                <!-- 几何形状 -->
                 <geometry>
-                    <box size="0.02 0.1 0.02"/>
+                    <!-- 长方体 长 宽 高 -->
+                    <box size="0.02 0.02 0.02"/>
                 </geometry>
+                <!-- 材质颜色 -->
                 <material name="black">
                     <color rgba="0.0 0.0 0.0 1.0"/>
@@ -18,5 +22,5 @@
                 <origin xyz="0 0 0" rpy="0 0 0"/>
                 <geometry>
-                    <box size="0.02 0.1 0.02"/>
+                    <box size="0.02 0.02 0.02"/>
                 </geometry>
                 <material name="black">
@@ -25,17 +29,11 @@
             </collision>
             <!-- 惯性描述 -->
-            <xacro:box_inertia m="0.1" w="0.02" h="0.1" d="0.02"/>
+            <xacro:box_inertia m="0.05" w="0.02" h="0.02" d="0.02"/>
         </link>
-        <link name="camera_optical_link"/>
         <!-- 机器人的关节,用于组成 -->
-        <joint name="camera_link_joint" type="fixed">
+        <joint name="imu_link_joint" type="fixed">
             <parent link="base_link"/>
-            <child link="camera_link"/>
+            <child link="imu_link"/>
             <origin xyz="${xyz}" rpy="0 0 0"/>
-        </joint>
-        <joint name="camera_optical_link_joint" type="fixed">
-            <parent link="camera_link"/>
-            <child link="camera_optical_link"/>
-            <origin xyz="0 0 0" rpy="${-pi/2} 0 ${-pi/2}"/>
         </joint>
     </xacro:macro>
