Commit message: Add auto patrol and Livox ROS driver packages for navigation and sensor integration

File: chap_navigation/src/demo_description/urdf/fishbot/fishbot.urdf.xacro (robot description, xacro)
@@ -6,4 +6,7 @@
     <xacro:property name="base_radius" value="0.1"/>
     <xacro:property name="wheel_radius" value="0.032"/>
+  <!-- base_link to livox_frame -->
+    <xacro:arg name="xyz" default="0.0 0.0 0.10" />
+    <xacro:arg name="rpy" default="0 0 0" />
     <!--基础部分 base_link-->
     <xacro:include filename="$(find demo_description)/urdf/fishbot/base.urdf.xacro"/>
@@ -19,6 +22,7 @@
     <xacro:include filename="$(find demo_description)/urdf/fishbot/plugins/gazebo_sensor_plugin.xacro"/>
     <xacro:include filename="$(find demo_description)/urdf/fishbot/fishbot.ros2_control.xacro"/>
+    <!-- <xacro:include filename="$(find demo_description)/urdf/fishbot/plugins/gazebo_laser_imu_plugin.xacro"/> -->
     <xacro:base_link length="${base_length}" radius="${base_radius}"/>
-    <xacro:imu_link xyz="0 0 0.02"/>
+    <xacro:imu_link xyz="0 0 0.04"/>
     <xacro:camera_link xyz="${base_radius} 0 0.075"/>
     <xacro:laser_link xyz="0.0 0 0.10"/>
@@ -30,3 +34,18 @@
     <xacro:gazebo_sensor_plugin/>
     <xacro:fishbot_ros2_control/>
+    <!-- mid360_imu plugin -->
+    <!-- https://github.com/ros-simulation/gazebo_ros_pkgs/wiki/ROS-2-Migration:-IMU-Sensors -->
+    <!-- <xacro:gazebo_imu_plugin/> -->
+    <!-- Livox-Mid360  -->
+    <!-- <xacro:include filename="$(find ros2_livox_simulation)/urdf/mid360.xacro" />
+    <xacro:mid360 name="livox_frame" parent="base_link" topic="/livox/lidar">
+        <origin xyz="$(arg xyz)" rpy="$(arg rpy)" />
+    </xacro:mid360> -->
+    <!-- 设置材质 -->
+    <gazebo reference="imu_link">
+        <material>Gazebo/BuildingFrame</material>
+    </gazebo>
+  <!-- <gazebo reference="livox_frame">
+    <material>Gazebo/LightBlueLaser</material>
+  </gazebo> -->
 </robot>

File: chap_navigation/src/demo_description/urdf/fishbot/plugins/gazebo_sensor_plugin.xacro (robot description, xacro)
@@ -16,14 +16,14 @@
                 <update_rate>5</update_rate>
                 <pose>0 0 0 0 0 0</pose>
-                <!-- 激光传感器配置 -->
-            <ray>
-                <!-- 设置扫描范围 -->
-                <scan>
-                    <horizontal>
-                        <samples>360</samples>
-                        <resolution>1.000000</resolution>
-                        <min_angle>0.000000</min_angle>
-                        <max_angle>6.280000</max_angle>
-                    </horizontal>
+								<!-- 激光传感器配置 -->
+                <ray>
+                    <!-- 设置扫描范围 -->
+                    <scan>
+                        <horizontal>
+                            <samples>360</samples>
+                            <resolution>1.000000</resolution>
+                            <min_angle>0.000000</min_angle>
+                            <max_angle>6.280000</max_angle>
+                        </horizontal>
                     </scan>
                     <!-- 设置扫描距离 -->
@@ -42,5 +42,5 @@
             </sensor>
         </gazebo>
-        <gazebo reference="imu_link">
+<gazebo reference="imu_link">
     <sensor name="imu_sensor" type="imu">
         <plugin name="imu_plugin" filename="libgazebo_ros_imu_sensor.so">

File: chap_simulation/src/demo_description/urdf/fishbot/fishbot.urdf.xacro (robot description, xacro)
@@ -6,4 +6,7 @@
     <xacro:property name="base_radius" value="0.1"/>
     <xacro:property name="wheel_radius" value="0.032"/>
+  <!-- base_link to livox_frame -->
+  <xacro:arg name="xyz" default="0.0 0.0 0.10" />
+  <xacro:arg name="rpy" default="0 0 0" />
     <!--基础部分 base_link-->
     <xacro:include filename="$(find demo_description)/urdf/fishbot/base.urdf.xacro"/>
@@ -30,3 +33,8 @@
     <xacro:gazebo_sensor_plugin/>
     <xacro:fishbot_ros2_control/>
+  <!-- Livox-Mid360  -->
+  <xacro:include filename="$(find ros2_livox_simulation)/urdf/mid360.xacro" />
+  <xacro:mid360 name="livox_frame" parent="base_link" topic="/livox/lidar">
+    <origin xyz="$(arg xyz)" rpy="$(arg rpy)" />
+  </xacro:mid360>
 </robot>
